Commit message: - Modified target_locator to optionally return position of cuboid as well as the sphere. - target_tracker now also publishes position of cuboid - target_follower now uses null space control to avoid hitting the cuboid - Changed limits of joint 2-4 angles to allow following target for more than 10 seconds

File: urdf/robot.urdf (robot description, URDF)
Before this commit: robot myrobot, 9 links, 8 joints
Joints:
- joint link0_to_link1: limit lower=-${pi/2} upper=${pi/2} effort=1000.0 velocity=5 -> lower=-${pi} upper=${pi} effort=1000.0 velocity=5
- joint link0_to_link1_2: limit lower=-${pi/2} upper=${pi/2} effort=1000.0 velocity=5 -> lower=-${pi} upper=${pi} effort=1000.0 velocity=5
- joint link1_to_link2: limit lower=-${pi/2} upper=${pi/2} effort=1000.0 velocity=5 -> lower=-${pi} upper=${pi} effort=1000.0 velocity=5
